Commit message: Added ft_sensor.

File: urdf/mybot.urdf (robot description, URDF)
Before this commit: robot arm, 10 links, 9 joints
Links:
- added link ft_sensor
Joints:
- added joint ft_sensor_joint: type fixed, parent hand, child ft_sensor, origin xyz=0 0 0.05 rpy=0 0 0
- joint wrist: limit (none) -> lower=-2.0 upper=2.0 effort=100 velocity=1; type continuous -> revolute
