Commit message: Some changes, trying out the controller.

File: src/robot_arm/urdf/arm.urdf (robot description, URDF)
Before this commit: robot robot_arm, 9 links, 8 joints
Links:
- removed link camera_link
- added link base
Joints:
- removed joint camera_joint
- added joint base_joint: type fixed, parent base, child base_link
